File: cad/MIDIcontroller/bank.kicad_sch (KiCad schematic)
At the start: 24 parts, among them U0 74HC595

Commit message: Added button on encoder
Parts:
- added C_ENSW1: 220n, Capacitor_Tantalum_SMD:CP_EIA-1608-08_AVX-J, symbol Device:C
- added R_ENSW1: 10k, Resistor_SMD:R_0805_2012Metric, symbol Device:R
Connections:
- net 5V: now also R_ENSW1.1
- net GND: now also SW_BANK1.S2, C_ENSW1.2
- net EN_S1: now reaches SW_BANK1.S1
- net EN_S1: now also C_ENSW1.1, R_ENSW1.2
- no-connect marks 0 -> 3
